File: cv-extractor-front-panel.kicad_pcb (KiCad board)
At the start: 2 copper layers, 40.3 x 128.5 mm, 5 parts

Commit message: havent been good about commits, its at V4 now
Parts:
- removed the ? at (100.0, 49.0)
- removed the ? at (100.0, 62.8)
- added ?: , MountingHole_7.0mm_PTV09, F.Cu at (100.0, 55.0)
- added ?: , MountingHole_7.0mm_PTV09, F.Cu at (100.0, 39.7)
- added ?: , MountingHole-mono-jack-thonk, F.Cu at (100.0, 27.5)
- added ?: , MountingHole-mono-jack-thonk, F.Cu at (100.0, 103.8)
- added REF**: MountingHole_3.2mm_M3, MountingHole:MountingHole_3.2mm_M3, F.Cu at (88.5, 61.0)
- added REF**: MountingHole_3.2mm_M3, MountingHole:MountingHole_3.2mm_M3, F.Cu at (111.5, 61.0)
- moved ? 40.3 mm to (100.0, 80.5)
Other:
- board text added: "CV Extractor V4"
- board text added: "CV Out"
- board text added: "Input Gain"
- board text added: "Output Gain"
- board text added: "Snappiness"
- board text added: "Wave In"
- board text removed: "CV Extractor V2 2021-10-29"
- board text removed: "Input"
- board text removed: "LPF Cutoff"
- board text removed: "Output"
Changed lines of the file:
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@@
   (general
     (thickness 1.6)
-    (drawings 8)
+    (drawings 10)
     (tracks 0)
     (zones 0)
-    (modules 5)
+    (modules 9)
     (nets 1)
   )
@@
     (uvia_drill 0.1)
   )
+  (module MountingHole:MountingHole_3.2mm_M3 (layer F.Cu)
+    (at 88.5 61)
+    (descr "Mounting Hole 3.2mm, no annular, M3")
+    (tags "mounting hole 3.2mm no annular m3")
+    (attr virtual)
+    (fp_text reference REF** (at 0 -4.2) (layer F.SilkS) hide
+      (effects (font (size 1 1) (thickness 0.15)))
+    )
+    (fp_text value MountingHole_3.2mm_M3 (at 0 4.2) (layer F.Fab) hide
+      (effects (font (size 1 1) (thickness 0.15)))
+    )
+    (fp_circle (center 0 0) (end 3.45 0) (layer F.CrtYd) (width 0.05))
+    (fp_circle (center 0 0) (end 3.2 0) (layer Cmts.User) (width 0.15))
+    (fp_text user %R (at 0.3 0) (layer F.Fab) hide
+      (effects (font (size 1 1) (thickness 0.15)))
+    )
+    (pad 1 np_thru_hole circle (at 0 0) (size 3.2 3.2) (drill 3.2) (layers *.Cu *.Mask))
+  )
+  (module MountingHole:MountingHole_3.2mm_M3 (layer F.Cu)
+    (at 111.5 61)
+    (descr "Mounting Hole 3.2mm, no annular, M3")
+    (tags "mounting hole 3.2mm no annular m3")
+    (attr virtual)
+    (fp_text reference REF** (at 0 -4.2) (layer F.SilkS) hide
+      (effects (font (size 1 1) (thickness 0.15)))
+    )
+    (fp_text value MountingHole_3.2mm_M3 (at 0 4.2) (layer F.Fab) hide
+      (effects (font (size 1 1) (thickness 0.15)))
+    )
+    (fp_text user %R (at 0.3 0) (layer F.Fab) hide
+      (effects (font (size 1 1) (thickness 0.15)))
+    )
+    (fp_circle (center 0 0) (end 3.2 0) (layer Cmts.User) (width 0.15))
+    (fp_circle (center 0 0) (end 3.45 0) (layer F.CrtYd) (width 0.05))
+    (pad 1 np_thru_hole circle (at 0 0) (size 3.2 3.2) (drill 3.2) (layers *.Cu *.Mask))
+  )
+  (module MountingHole_7.0mm_PTV09 (layer F.Cu)
+    (at 100 55)
+    (descr "Mounting Hole 6.4mm, no annular, M6")
+    (tags "mounting hole 6.4mm no annular m6")
+    (attr virtual)
+    (fp_text reference "" (at 0 -7.4) (layer F.SilkS) hide
+      (effects (font (size 1 1) (thickness 0.15)))
+    )
+    (fp_text value "" (at 0 7.4) (layer F.Fab) hide
+      (effects (font (size 1 1) (thickness 0.15)))
+    )
+    (fp_circle (center 0 0) (end 7.4 0) (layer Cmts.User) (width 0.15))
+    (fp_circle (center 0 0) (end 7.65 0) (layer F.CrtYd) (width 0.05))
+    (fp_text user %R (at 0.3 0) (layer F.Fab) hide
+      (effects (font (size 1 1) (thickness 0.15)))
+    )
+    (pad "" np_thru_hole circle (at 0 0) (size 7 7) (drill 7) (layers *.Cu *.Mask))
+  )
+  (module MountingHole_7.0mm_PTV09 (layer F.Cu)
+    (at 100 39.7)
+    (descr "Mounting Hole 6.4mm, no annular, M6")
+    (tags "mounting hole 6.4mm no annular m6")
+    (attr virtual)
+    (fp_text reference "" (at 0 -7.4) (layer F.SilkS) hide
+      (effects (font (size 1 1) (thickness 0.15)))
+    )
+    (fp_text value "" (at 0 7.4) (layer F.Fab) hide
+      (effects (font (size 1 1) (thickness 0.15)))
+    )
+    (fp_circle (center 0 0) (end 7.4 0) (layer Cmts.User) (width 0.15))
+    (fp_circle (center 0 0) (end 7.65 0) (layer F.CrtYd) (width 0.05))
+    (fp_text user %R (at 0.3 0) (layer F.Fab) hide
+      (effects (font (size 1 1) (thickness 0.15)))
+    )
+    (pad "" np_thru_hole circle (at 0 0) (size 7 7) (drill 7) (layers *.Cu *.Mask))
+  )
+  (module MountingHole-dual-pot-P120 (layer F.Cu)
+    (at 100 80.55)
+    (fp_text reference "" (at 0.3 -5.9) (layer F.SilkS)
+      (effects (font (size 1 1) (thickness 0.15)))
+    )
+    (fp_text value "" (at -0.127 -15.24) (layer F.Fab)
+      (effects (font (size 1 1) (thickness 0.15)))
+    )
+    (pad 1 thru_hole circle (at 0 -10) (size 6.5 6.5) (drill 6.3) (layers *.Cu *.Mask))
+  )
   (module MountingHole-mono-jack-thonk (layer F.Cu)
-    (at 100 49 180)
+    (at 100 27.5 180)
     (fp_text reference "" (at -0.1 -2.7 180) (layer F.SilkS)
       (effects (font (size 1 1) (thickness 0.15)))
@@
       (effects (font (size 1 1) (thickness 0.15)))
     )
-    (pad "" thru_hole circle (at 0 0 180) (size 3.5 3.5) (drill 3) (layers *.Cu *.Mask))
-  )
-  (module MountingHole-dual-pot-P120 (layer F.Cu)
-    (at 100 40.2)
-    (fp_text reference "" (at 0.3 -5.9) (layer F.SilkS)
-      (effects (font (size 1 1) (thickness 0.15)))
-    )
-    (fp_text value "" (at -0.127 -15.24) (layer F.Fab)
-      (effects (font (size 1 1) (thickness 0.15)))
-    )
-    (pad 1 thru_hole circle (at 0 -10) (size 6.5 6.5) (drill 6.3) (layers *.Cu *.Mask))
+    (pad "" thru_hole circle (at 0 0 180) (size 7 7) (drill 6.5) (layers *.Cu *.Mask))
   )
   (module MountingHole-mono-jack-thonk (layer F.Cu)
-    (at 100 62.75 180)
+    (at 100 103.75 180)
     (fp_text reference "" (at -0.1 -2.7 180) (layer F.SilkS)
       (effects (font (size 1 1) (thickness 0.15)))
@@
       (effects (font (size 1 1) (thickness 0.15)))
     )
-    (pad "" thru_hole circle (at 0 0 180) (size 3.5 3.5) (drill 3) (layers *.Cu *.Mask))
+    (pad "" thru_hole circle (at 0 0 180) (size 7 7) (drill 6.5) (layers *.Cu *.Mask))
   )
   (module MountingHole_M3_slot (layer F.Cu)
@@
       (effects (font (size 1 1) (thickness 0.15)))
     )
-    (fp_circle (center 0 0) (end 3.45 0) (layer F.CrtYd) (width 0.05))
-    (fp_circle (center 0 0) (end 3.2 0) (layer Cmts.User) (width 0.15))
+    (fp_circle (center 0 0) (end 3.2 0) (layer Cmts.User) (width 0.15))
+    (fp_circle (center 0 0) (end 3.45 0) (layer F.CrtYd) (width 0.05))
     (fp_text user %R (at 0.3 0) (layer F.Fab) hide
       (effects (font (size 1 1) (thickness 0.15)))
@@
       (effects (font (size 1 1) (thickness 0.15)))
     )
-    (fp_circle (center 0 0) (end 3.45 0) (layer F.CrtYd) (width 0.05))
-    (fp_circle (center 0 0) (end 3.2 0) (layer Cmts.User) (width 0.15))
+    (fp_circle (center 0 0) (end 3.2 0) (layer Cmts.User) (width 0.15))
+    (fp_circle (center 0 0) (end 3.45 0) (layer F.CrtYd) (width 0.05))
     (fp_text user %R (at 0.3 0) (layer F.Fab) hide
       (effects (font (size 1 1) (thickness 0.15)))
@@
     (pad "" np_thru_hole oval (at 0 0) (size 4 3.200001) (drill oval 4 3.200001) (layers *.Cu *.Mask))
   )
-  (gr_text "CV Extractor V2\n2021-10-29" (at 100 16.2) (layer F.SilkS)
-    (effects (font (size 1.5 1.5) (thickness 0.3)))
-  )
-  (gr_text Output (at 99.95 59.275) (layer F.SilkS)
-    (effects (font (size 1.5 1.5) (thickness 0.3)))
-  )
-  (gr_text Input (at 99.975 45.25) (layer F.SilkS)
-    (effects (font (size 1.5 1.5) (thickness 0.3)))
-  )
-  (gr_text "LPF Cutoff" (at 100 25.25) (layer F.SilkS)
-    (effects (font (size 1.5 1.5) (thickness 0.3)))
+  (gr_text "CV Extractor V4" (at 100 15.45) (layer F.SilkS)
+    (effects (font (size 3 3) (thickness 0.3)))
+  )
+  (gr_text "CV Out" (at 100.15 97.75) (layer F.SilkS)
+    (effects (font (size 2 2) (thickness 0.3)))
+  )
+  (gr_text Snappiness (at 100 64.575) (layer F.SilkS)
+    (effects (font (size 2 2) (thickness 0.3)))
+  )
+  (gr_text "Output Gain" (at 100 48.825) (layer F.SilkS)
+    (effects (font (size 2 2) (thickness 0.3)))
+  )
+  (gr_text "Input Gain" (at 100 33.575) (layer F.SilkS)
+    (effects (font (size 2 2) (thickness 0.3)))
+  )
+  (gr_text "Wave In" (at 100 22.15) (layer F.SilkS)
+    (effects (font (size 2 2) (thickness 0.3)))
   )
   (gr_line (start 79.85 134.25) (end 79.85 5.75) (layer Edge.Cuts) (width 0.1))
